File: Barometer 022.brd (EAGLE design)
At the start: 62.5 x 41.9 mm, 97 parts, among them IC1 MIC5225-3.3v, IC2 TPS5410, Q2 SI2306-TP, Q3 SI2306-TP, Q6 BSP170P, Q7 KST2907, U1 Tiny85-20-SMT, U2 DAC8574, U3 TPS55340RTER, U4 MAX3221, U5 ICP-20100, U6 XTR111AIDRCR, U7 LTC4365ITS8TRPBF, X1 1751264, X2 1751248

Commit message: x
Parts:
- added D4, D5, D7: SMBJ6.0CA, SMBJ6.0CA:DIOM4336X265N
- added D6: SMBJ24CA, SMBJ24CA:DIOM4336X265N
- added R23: 100, microbuilder:0603
- added R24, R25, R26, R27: 10k, microbuilder:0603
- added R28, R29: 20k, microbuilder:0603
- added R30: 120, microbuilder:0603
- added SJ2, SJ8, SJ9: SOLDERJUMPERTRACE, SparkFun-Retired-0:SJ_2S-TRACE
- added SJ3: (no value), jumper:SJ_2
- added U8: LTC2850, LTC_By_element14_Batch_1:SOIC127P600X175-8N
- C1, C10, C12, C15, C16, C17, C2, C3, C4, C5, C6, C7, C8, C9: device microbuilder:0603 -> microbuilder:0603@1
- C11: device microbuilder:0805 -> microbuilder:0805@1
- C13, C14, C18, C19: device microbuilder:1206 -> microbuilder:1206@1
- moved TP5 1.71 mm to (30.7, 22.5)
- moved TP12 0.89 mm to (31.4, 9.78)
- moved TP1 0.32 mm to (24.1, 35.2)
- renumbered PAD10 to PAD1, PAD11 to PAD3, PAD12 to PAD5, PAD7 to PAD6, PAD8 to PAD4, PAD9 to PAD2, Q7 to Q5, SJ13 to SJ10, SJ14 to SJ11, SJ16 to SJ12, U$8 to U$4
Connections:
- new net 485EN: R25.1, R26.1, SJ2.2, U8.2, U8.3
- new net A: R28.1, R30.2, SJ3.1, U8.6
- new net A-GND: R23.2, X1.1
- new net B: R29.1, R30.1, SJ8.2, U8.7
- new net D-OUT-1: D5.1, SJ8.1, SJ9.1, X1.4
- new net D-OUT-2: D4.1, SJ3.2, X1.3
- net +3V3: now also R24.2, R25.2, R26.2, R27.2, R28.2, U8.8
- net B1: now also SJ2.1
- net DIN: now also R27.1, U8.4
- net DOUT: now also SJ3.3; no longer X1.3
- net GND: now also D4.2, D5.2, D6.1, D7.2, R23.1, R29.2, U8.5; no longer X1.1
- net LOAD: now also D6.2
- net RIN: now also SJ9.2; no longer X1.4
- net ROUT: now also R24.1, U8.1
- net V-OUT-2: now also D7.1
Routing:
- net 485EN: track 0.00 -> 90.2 mm, vias 0 -> 2
- net ROUT: track 14.4 -> 86.9 mm, vias 1 -> 4
- net D-OUT-2: track 0.00 -> 67.1 mm, vias 0 -> 1
- net D-OUT-1: track 0.00 -> 58.9 mm, vias 0 -> 1
- net DOUT: track 40.5 -> 87.8 mm
- net DIN: track 15.9 -> 59.9 mm, vias 1 -> 4
- net B: track 0.00 -> 41.1 mm, vias 0 -> 2
- net A: track 0.00 -> 34.1 mm, vias 0 -> 1
- net +3V3: track 111.6 -> 140.8 mm
- net B1: track 2.29 -> 18.8 mm, vias 0 -> 1
- net V-OUT-2: track 14.4 -> 21.8 mm
- net LOAD: track 5.45 -> 12.2 mm
- net RIN: track 37.4 -> 32.5 mm
- net A-GND: track 0.00 -> 2.94 mm
- net SCL_3V3: track 59.8 -> 61.7 mm
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Other:
- board text added: "D4"
- board text added: "D5"
- board text added: "D6"
- board text added: "D7"
- board text added: "Q5"
- board text added: "R23"
- board text added: "R24"
- board text added: "R25"
- board text added: "R26"
- board text added: "R27"
- board text added: "R28"
- board text added: "R29"
- board text added: "R30"
- board text added: "RS232"
- board text added: "RS485"
- board text added: "RX/B"
- board text added: "SGS Weather & Environmental Systems SGB022 v2.0 rev. D"
- board text added: "SJ10"
- board text added: "SJ11"
- board text added: "SJ12"
- board text added: "SJ2"
- board text added: "SJ3"
- board text added: "SJ8"
- board text added: "SJ9"
- board text added: "TX/A"
- board text added: "U8"
- board text removed: "Q7"
- board text removed: "RX"
- board text removed: "SGS Weather & Environmental Systems SGB 022 rev. I"
- board text removed: "SJ13"
- board text removed: "SJ14"
- board text removed: "SJ16"
- board text removed: "TX"
