File: Barometer 022.sch (EAGLE design)
At the start: 97 parts, among them IC1 MIC5225-3.3v, IC2 TPS5410, Q2 SI2306-TP, Q3 SI2306-TP, Q6 BSP170P, Q7 KST2907, U1 Tiny85-20-SMT, U2 DAC8574, U3 TPS55340RTER, U4 MAX3221, U5 ICP-20100, U6 XTR111AIDRCR, U7 LTC4365ITS8TRPBF, X1 1751264, X2 1751248

Commit message: x
Parts:
- added D4, D5, D7: SMBJ6.0CA, SMBJ6.0CA:SMBJ6.0CA
- added D6: SMBJ24CA, SMBJ24CA:SMBJ24CA
- added R23: 100, microbuilder:RESISTOR0603
- added R24, R25, R26, R27: 10k, microbuilder:RESISTOR0603
- added R28, R29: 20k, microbuilder:RESISTOR0603
- added R30: 120, microbuilder:RESISTOR0603
- added SJ2, SJ8, SJ9: SOLDERJUMPERTRACE, SparkFun-Retired-0:SOLDERJUMPERTRACE
- added SJ3: (no value), jumper:SJ2W
- added U8: LTC2850, LTC_By_element14_Batch_1:LTC2850IS8PBF
- renumbered PAD10 to PAD1, PAD11 to PAD3, PAD12 to PAD5, PAD7 to PAD6, PAD8 to PAD4, PAD9 to PAD2, Q7 to Q5, SJ13 to SJ10, SJ14 to SJ11, SJ16 to SJ12, U$8 to U$4
Connections:
- new net 485EN: R25.1, R26.1, SJ2.2, U8.DE, U8.~RE
- new net A: R28.1, R30.2, SJ3.1, U8.A
- new net A-GND: R23.2, X1-1.K
- new net B: R29.1, R30.1, SJ8.2, U8.B
- new net D-OUT-1: D5.1, SJ8.1, SJ9.1, X1-4.K
- new net D-OUT-2: D4.1, SJ3.2, X1-3.K
- net +3V3: now also R24.2, R25.2, R26.2, R27.2, R28.2, U8.VCC
- net B1: now also SJ2.1
- net DIN: now also R27.1, U8.DI
- net DOUT: now also SJ3.3; no longer X1-3.K
- net GND: now also D4.2, D5.2, D6.1, D7.2, R23.1, R29.2, U8.GND; no longer X1-1.K
- net LOAD: now also D6.2
- net RIN: now also SJ9.2; no longer X1-4.K
- net ROUT: now also R24.1, U8.RO
- net V-OUT-2: now also D7.1
